File: ecp-v-wireless/MISC-IO.kicad_sch (KiCad schematic)
At the start: 1 part, among them U2 LFE5U-85F-6BG381x

Commit message: Continued schematic work
Signed-off-by: Michael Welling <mwelling79@gmail.com>
Parts:
- added C20, C21, C22: 0.1uf, Capacitor_SMD:C_0402_1005Metric, symbol Device:C_Small
- added D3: CLX6F-FKC, LED_SMD:LED_RGB_PLCC-6, symbol emeb_library:LED_BGR
- added JP2, JP3, JP4: SolderJumper_3_Bridged12, Jumper:SolderJumper-3_P1.3mm_Bridged12_RoundedPad1.0x1.5mm, symbol Jumper:SolderJumper_3_Bridged12
- added PMOD1, PMOD2, PMOD3: CONN_02X06, Connector_PinSocket_2.54mm:PinSocket_2x06_P2.54mm_Vertical, symbol Connector_Generic:Conn_02x06_Odd_Even
Connections:
- new net +3V3: D3.4 (BA), D3.5 (GA), D3.6 (RA), JP2.1 (A), JP3.1 (A), JP4.1 (A)
- new net +4V: JP2.3 (B), JP3.3 (B), JP4.3 (B)
- new net GND: C20.2, C21.2, C22.2, PMOD1.10 (Pin_10), PMOD1.9 (Pin_9), PMOD2.10 (Pin_10), PMOD2.9 (Pin_9), PMOD3.10 (Pin_10), PMOD3.9 (Pin_9)
- new net VJ5: C22.1, JP3.2 (C), PMOD3.11 (Pin_11), PMOD3.12 (Pin_12)
- new net VJ6: C21.1, JP2.2 (C), PMOD2.11 (Pin_11), PMOD2.12 (Pin_12)
- new net VJ7: C20.1, JP4.2 (C), PMOD1.11 (Pin_11), PMOD1.12 (Pin_12)
Other:
- note added: "Das blinkenled."
- note added: "PMOD Supply Select Default to 3.3V"
- note removed: "- ADD PMOD INTERFACE"
- note removed: "- ADD RGB LED"
- moved on the sheet: U2B, U2C, U2D, U2E, U2F, U2G, U2H
