File: ecp-v-wireless/POWER.kicad_sch (KiCad schematic)
At the start: 37 parts, among them Q1 DMP1045U-7, U2 LFE5U-85F-6BG381x, U4 TLV62569DRL, U5 TLV62569DRL, U6 TLV713285PDBV, U7 MCP73831-2-OT

Commit message: Continued schematic work
Signed-off-by: Michael Welling <mwelling79@gmail.com>
Parts:
- C10, C11, C12, C13, C14, C15, C16, C17, C4, C5, C6, C7, C8, C9: symbol Device:C -> Device:C_Small
- R9: value 84k5 -> 84.5k
Other:
- note added: "BATTERY MANAGEMENT CIRCUIT COPIED FROM ICE-V WIRELESS"
- note added: "POWER SUPPLIES COPIED FROM ICEBREAKER++/ICECRUSHER DESIGN"
