File: ecp-v-wireless/ecp-v-wireless.kicad_pcb (KiCad board)
At the start: 2 copper layers, 81.7 x 31.8 mm, 56 parts, among them J1 USB_C_Receptacle_USB2.0_16P, Q1 DMP1045U-7, SW1 SW_Push, SW2 SW_Push, U1 ESP32-S3-MINI-1, U2 LFE5U-85F-6BG381x, U3 DRTR5V0U4S, U4 TLV62569DRL, U5 TLV62569DRL, U6 TLV713285PDBV, U7 MCP73831-2-OT

Commit message: Continued schematic work
Signed-off-by: Michael Welling <mwelling79@gmail.com>
Parts:
- added C20: 0.1uf, Capacitor_SMD:C_0402_1005Metric, F.Cu at (134.8, 61.5)
- added C21: 0.1uf, Capacitor_SMD:C_0402_1005Metric, F.Cu at (134.8, 63.5)
- added C22: 0.1uf, Capacitor_SMD:C_0402_1005Metric, F.Cu at (134.8, 65.4)
- added D3: CLX6F-FKC, LED_SMD:LED_RGB_PLCC-6, F.Cu at (157.3, 60.0)
- added JP2: SolderJumper_3_Bridged12, Jumper:SolderJumper-3_P1.3mm_Bridged12_RoundedPad1.0x1.5mm, F.Cu at (136.2, 50.8)
- added JP3: SolderJumper_3_Bridged12, Jumper:SolderJumper-3_P1.3mm_Bridged12_RoundedPad1.0x1.5mm, F.Cu at (136.2, 54.6)
- added JP4: SolderJumper_3_Bridged12, Jumper:SolderJumper-3_P1.3mm_Bridged12_RoundedPad1.0x1.5mm, F.Cu at (136.2, 58.4)
- added PMOD1: CONN_02X06, Connector_PinSocket_2.54mm:PinSocket_2x06_P2.54mm_Vertical, F.Cu at (116.8, 51.3)
- added PMOD2: CONN_02X06, Connector_PinSocket_2.54mm:PinSocket_2x06_P2.54mm_Vertical, F.Cu at (124.0, 51.3)
- added PMOD3: CONN_02X06, Connector_PinSocket_2.54mm:PinSocket_2x06_P2.54mm_Vertical, F.Cu at (131.1, 51.3)
- R9: value 84k5 -> 84.5k
