File: ecp-v-wireless/ecp-v-wireless.kicad_sch (KiCad schematic)
At the start: 0 parts

Commit message: Continued schematic work
Signed-off-by: Michael Welling <mwelling79@gmail.com>
Changed lines of the file:
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@@
 	(text_box "ESP32-S3 MCU"
 		(exclude_from_sim no)
-		(at 130.81 68.58 0)
+		(at 109.22 68.58 0)
 		(size 22.86 13.97)
 		(margins 0.9525 0.9525 0.9525 0.9525)
@@
 	(text_box "1.1V\nBUCK"
 		(exclude_from_sim no)
-		(at 138.43 116.84 0)
+		(at 116.84 116.84 0)
 		(size 8.89 5.9929)
 		(margins 0.9525 0.9525 0.9525 0.9525)
@@
 	(text_box "USB-C"
 		(exclude_from_sim no)
-		(at 113.03 68.58 0)
+		(at 91.44 68.58 0)
 		(size 8.89 5.08)
 		(margins 0.9525 0.9525 0.9525 0.9525)
@@
 	(text_box "LiPO\nCONN"
 		(exclude_from_sim no)
-		(at 113.03 99.4171 0)
+		(at 91.44 99.4171 0)
 		(size 8.89 5.9929)
 		(margins 0.9525 0.9525 0.9525 0.9525)
@@
 	(text_box "3.3V\nBUCK"
 		(exclude_from_sim no)
-		(at 138.43 107.95 0)
+		(at 116.84 107.95 0)
+		(size 8.89 5.9929)
+		(margins 0.9525 0.9525 0.9525 0.9525)
+		(stroke
+			(width 0)
+			(type solid)
+		)
+		(fill
+			(type none)
+		)
+		(effects
+			(font
+				(size 1.27 1.27)
+			)
+		)
+	)
+	(text_box "RGB LED"
+		(exclude_from_sim no)
+		(at 184.15 68.58 0)
+		(size 8.89 5.9929)
+		(margins 0.9525 0.9525 0.9525 0.9525)
+		(stroke
+			(width 0)
+			(type solid)
+		)
+		(fill
+			(type none)
+		)
+		(effects
+			(font
+				(size 1.27 1.27)
+			)
+		)
+	)
+	(text_box "PMOD2"
+		(exclude_from_sim no)
+		(at 195.58 76.2 0)
 		(size 8.89 5.9929)
 		(margins 0.9525 0.9525 0.9525 0.9525)
@@
 	(text_box "2.5V\nLDO"
 		(exclude_from_sim no)
-		(at 138.43 124.8171 0)
+		(at 116.84 124.8171 0)
+		(size 8.89 5.9929)
+		(margins 0.9525 0.9525 0.9525 0.9525)
+		(stroke
+			(width 0)
+			(type solid)
+		)
+		(fill
+			(type none)
+		)
+		(effects
+			(font
+				(size 1.27 1.27)
+			)
+		)
+	)
+	(text_box "PMOD1"
+		(exclude_from_sim no)
+		(at 195.58 68.58 0)
 		(size 8.89 5.9929)
 		(margins 0.9525 0.9525 0.9525 0.9525)
@@
 	(text_box "ECP5 FPGA\nLFE5U-85F-6BG381x"
 		(exclude_from_sim no)
-		(at 161.29 68.58 0)
+		(at 138.43 81.28 0)
 		(size 22.86 13.97)
 		(margins 0.9525 0.9525 0.9525 0.9525)
@@
 		)
 	)
+	(text_box "PMOD3"
+		(exclude_from_sim no)
+		(at 195.58 83.82 0)
+		(size 8.89 5.9929)
+		(margins 0.9525 0.9525 0.9525 0.9525)
+		(stroke
+			(width 0)
+			(type solid)
+		)
+		(fill
+			(type none)
+		)
+		(effects
+			(font
+				(size 1.27 1.27)
+			)
+		)
+	)
 	(text_box "LIPO BATTERY MGMT"
 		(exclude_from_sim no)
-		(at 130.81 91.44 0)
+		(at 109.22 91.44 0)
 		(size 22.86 13.97)
 		(margins 0.9525 0.9525 0.9525 0.9525)
@@
 	(polyline
 		(pts
-			(xy 121.92 71.12) (xy 125.73 71.12)
-		)
-		(stroke
-			(width 0)
-			(type default)
-		)
-	)
-	(polyline
-		(pts
-			(xy 125.73 92.71) (xy 125.73 76.2)
-		)
-		(stroke
-			(width 0)
-			(type default)
-		)
-	)
-	(polyline
-		(pts
-			(xy 130.81 92.71) (xy 125.73 92.71)
-		)
-		(stroke
-			(width 0)
-			(type default)
-		)
-	)
-	(polyline
-		(pts
-			(xy 121.92 102.87) (xy 130.81 102.87)
-		)
-		(stroke
-			(width 0)
-			(type default)
-		)
-	)
-	(polyline
-		(pts
-			(xy 125.73 71.12) (xy 125.73 76.2)
-		)
-		(stroke
-			(width 0)
-			(type default)
-		)
-	)
-	(polyline
-		(pts
-			(xy 125.73 76.2) (xy 130.81 76.2)
+			(xy 100.33 71.12) (xy 104.14 71.12)
+		)
+		(stroke
+			(width 0)
+			(type default)
+		)
+	)
+	(polyline
+		(pts
+			(xy 104.14 92.71) (xy 104.14 76.2)
+		)
+		(stroke
+			(width 0)
+			(type default)
+		)
+	)
+	(polyline
+		(pts
+			(xy 109.22 92.71) (xy 104.14 92.71)
+		)
+		(stroke
+			(width 0)
+			(type default)
+		)
+	)
+	(polyline
+		(pts
+			(xy 100.33 102.87) (xy 109.22 102.87)
+		)
+		(stroke
+			(width 0)
+			(type default)
+		)
+	)
+	(polyline
+		(pts
+			(xy 104.14 71.12) (xy 104.14 76.2)
+		)
+		(stroke
+			(width 0)
+			(type default)
+		)
+	)
+	(polyline
+		(pts
+			(xy 104.14 76.2) (xy 109.22 76.2)
 		)
 		(stroke
@@
 	)
 	(sheet
-		(at 102.87 66.04)
+		(at 81.28 66.04)
 		(size 55.88 21.59)
 		(exclude_from_sim no)
@@
 		)
 		(property "Sheetname" "ESP32-S3"
-			(at 102.87 65.3284 0)
+			(at 81.28 65.3284 0)
 			(show_name no)
 			(do_not_autoplace no)
@@
 		)
 		(property "Sheetfile" "ESP32-S3.kicad_sch"
-			(at 132.842 63.754 0)
+			(at 111.252 63.754 0)
 			(show_name no)
 			(do_not_autoplace no)
@@
 	)
 	(sheet
-		(at 160.02 66.04)
-		(size 48.26 67.31)
+		(at 162.56 66.04)
+		(size 45.72 25.4)
 		(exclude_from_sim no)
 		(in_bom yes)
@@
 		)
 		(property "Sheetname" "MISC-IO"
-			(at 160.02 65.3284 0)
+			(at 162.56 65.3284 0)
 			(show_name no)
 			(do_not_autoplace no)
@@
 		)
 		(property "Sheetfile" "MISC-IO.kicad_sch"
-			(at 184.15 64.262 0)
+			(at 184.912 64.262 0)
 			(show_name no)
 			(do_not_autoplace no)
@@
 	)
 	(sheet
-		(at 102.87 90.17)
+		(at 81.28 90.17)
 		(size 55.88 43.18)
 		(exclude_from_sim no)
@@
 		)
 		(property "Sheetname" "POWER"
-			(at 102.87 89.4584 0)
+			(at 81.28 89.4584 0)
 			(show_name no)
 			(do_not_autoplace no)
@@
 		)
 		(property "Sheetfile" "POWER.kicad_sch"
-			(at 136.144 88.138 0)
+			(at 114.554 88.138 0)
 			(show_name no)
 			(do_not_autoplace no)
@@
 			(project "ecp-v-wireless"
 				(path "/eae84144-7f2d-46b9-a4e0-986cae4bd3c1"
-					(page "5")
-				)
-			)
+					(page "3")
+				)
+			)
