File: hardware/ESP32-S3.kicad_sch (KiCad schematic)
At the start: 15 parts, among them J1 USB_C_Receptacle_USB2.0_16P, SW1 SW_Push, SW2 SW_Push, U1 ESP32-S3-MINI-1, U2 LFE5U-85F-6BG381x, U3 DRTR5V0U4S

Commit message: Rando updates
Signed-off-by: Michael Welling <mwelling79@gmail.com>
Connections:
- net TCK: now reaches U1.5 (IO1)
- net TCK: now also U2.T5 (TCK)
- net TMS: now reaches U1.6 (IO2)
- net TMS: now also U2.U5 (TMS)
- net TDI: now reaches U1.7 (IO3)
- net TDI: now also U2.R5 (TDI)
- net TDO: now reaches U1.8 (IO4)
- net TDO: now also U2.V4 (TDO)
Changed lines of the file:
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@@
+	(wire
+		(pts
+			(xy 165.1 138.43) (xy 161.29 138.43)
+		)
+		(stroke
+			(width 0)
+			(type default)
+		)
+	)
 	(wire
 		(pts
@@
 	(wire
 		(pts
+			(xy 110.49 59.69) (xy 119.38 59.69)
+		)
+		(stroke
+			(width 0)
+			(type default)
+		)
+	)
+	(wire
+		(pts
 			(xy 196.85 34.29) (xy 207.01 34.29)
 		)
@@
 	(wire
 		(pts
+			(xy 165.1 140.97) (xy 161.29 140.97)
+		)
+		(stroke
+			(width 0)
+			(type default)
+		)
+	)
+	(wire
+		(pts
 			(xy 118.11 40.64) (xy 118.11 39.37)
 		)
@@
 	(wire
 		(pts
+			(xy 110.49 67.31) (xy 119.38 67.31)
+		)
+		(stroke
+			(width 0)
+			(type default)
+		)
+	)
+	(wire
+		(pts
+			(xy 110.49 64.77) (xy 119.38 64.77)
+		)
+		(stroke
+			(width 0)
+			(type default)
+		)
+	)
+	(wire
+		(pts
 			(xy 60.96 67.31) (xy 68.58 67.31)
 		)
@@
 	(wire
 		(pts
+			(xy 110.49 62.23) (xy 119.38 62.23)
+		)
+		(stroke
+			(width 0)
+			(type default)
+		)
+	)
+	(wire
+		(pts
 			(xy 76.2 52.07) (xy 60.96 52.07)
 		)
@@
 	(wire
 		(pts
+			(xy 165.1 135.89) (xy 161.29 135.89)
+		)
+		(stroke
+			(width 0)
+			(type default)
+		)
+	)
+	(wire
+		(pts
 			(xy 170.18 62.23) (xy 177.165 62.23)
+		)
+		(stroke
+			(width 0)
+			(type default)
+		)
+	)
+	(wire
+		(pts
+			(xy 165.1 133.35) (xy 161.29 133.35)
 		)
 		(stroke
@@
 		)
 	)
+	(label "TCK"
+		(at 165.1 135.89 0)
+		(effects
+			(font
+				(size 1.27 1.27)
+			)
+			(justify left bottom)
+		)
+	)
 	(label "RAW_D_P"
 		(at 196.85 54.61 0)
@@
 		)
 	)
+	(label "TCK"
+		(at 110.49 59.69 0)
+		(effects
+			(font
+				(size 1.27 1.27)
+			)
+			(justify left bottom)
+		)
+	)
+	(label "TDI"
+		(at 110.49 64.77 0)
+		(effects
+			(font
+				(size 1.27 1.27)
+			)
+			(justify left bottom)
+		)
+	)
+	(label "TMS"
+		(at 110.49 62.23 0)
+		(effects
+			(font
+				(size 1.27 1.27)
+			)
+			(justify left bottom)
+		)
+	)
 	(label "USB_D_N"
 		(at 160.02 59.69 180)
@@
 		)
 	)
+	(label "TDI"
+		(at 165.1 138.43 0)
+		(effects
+			(font
+				(size 1.27 1.27)
+			)
+			(justify left bottom)
+		)
+	)
 	(label "NRST"
 		(at 110.49 52.07 0)
 		(effects
 			(font
+				(size 1.27 1.27)
+			)
+			(justify left bottom)
+		)
+	)
+	(label "TDO"
+		(at 165.1 133.35 0)
+		(effects
+			(font
+				(size 1.27 1.27)
+			)
+			(justify left bottom)
+		)
+	)
+	(label "TMS"
+		(at 165.1 140.97 0)
+		(effects
+			(font
+				(size 1.27 1.27)
+			)
+			(justify left bottom)
+		)
+	)
+	(label "TDO"
+		(at 110.49 67.31 0)
+		(effects
+			(font
