File: hardware/POWER.kicad_sch (KiCad schematic)
At the start: 37 parts, among them Q1 DMP1045U-7, U2 LFE5U-85F-6BG381x, U4 TLV62569DRL, U5 TLV62569DRL, U6 TLV713285PDBV, U7 MCP73831-2-OT

Commit message: Rando updates
Signed-off-by: Michael Welling <mwelling79@gmail.com>
Other:
- moved on the sheet: C13, C6, C7, C9
