File: hardware/ecp-v-wireless.kicad_pcb (KiCad board)
At the start: 2 copper layers, 81.7 x 31.8 mm, 66 parts, among them J1 USB_C_Receptacle_USB2.0_16P, Q1 DMP1045U-7, SW1 SW_Push, SW2 SW_Push, U1 ESP32-S3-MINI-1, U2 LFE5U-85F-6BG381x, U3 DRTR5V0U4S, U4 TLV62569DRL, U5 TLV62569DRL, U6 TLV713285PDBV, U7 MCP73831-2-OT

Commit message: Rando updates
Signed-off-by: Michael Welling <mwelling79@gmail.com>
Connections:
- U1 pad 5: unconnected-(U1-IO1-Pad5) -> /ESP32-S3/TCK
- U1 pad 6: unconnected-(U1-IO2-Pad6) -> /ESP32-S3/TMS
- U1 pad 7: unconnected-(U1-IO3-Pad7) -> /ESP32-S3/TDI
- U1 pad 8: unconnected-(U1-IO4-Pad8) -> /ESP32-S3/TDO
- U2 pad R5: unconnected-(U2I-TDI-PadR5) -> /ESP32-S3/TDI
- U2 pad T5: unconnected-(U2I-TCK-PadT5) -> /ESP32-S3/TCK
- U2 pad U5: unconnected-(U2I-TMS-PadU5) -> /ESP32-S3/TMS
- U2 pad V4: unconnected-(U2I-TDO-PadV4) -> /ESP32-S3/TDO
Changed lines of the file:
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@@
 			(property pad_prop_bga)
 			(layers "F.Cu" "F.Mask" "F.Paste")
-			(net "unconnected-(U2I-TDI-PadR5)")
+			(net "/ESP32-S3/TDI")
 			(pinfunction "TDI_R5")
 			(pintype "input")
@@
 			(property pad_prop_bga)
 			(layers "F.Cu" "F.Mask" "F.Paste")
-			(net "unconnected-(U2I-TCK-PadT5)")
+			(net "/ESP32-S3/TCK")
 			(pinfunction "TCK_T5")
 			(pintype "input")
@@
 			(property pad_prop_bga)
 			(layers "F.Cu" "F.Mask" "F.Paste")
-			(net "unconnected-(U2I-TMS-PadU5)")
+			(net "/ESP32-S3/TMS")
 			(pinfunction "TMS_U5")
 			(pintype "input")
@@
 			(property pad_prop_bga)
 			(layers "F.Cu" "F.Mask" "F.Paste")
-			(net "unconnected-(U2I-TDO-PadV4)")
+			(net "/ESP32-S3/TDO")
 			(pinfunction "TDO_V4")
 			(pintype "output")
@@
 			(size 0.8 0.4)
 			(layers "F.Cu" "F.Mask" "F.Paste")
-			(net "unconnected-(U1-IO1-Pad5)")
+			(net "/ESP32-S3/TCK")
 			(pinfunction "IO1_5")
 			(pintype "bidirectional")
@@
 			(size 0.8 0.4)
 			(layers "F.Cu" "F.Mask" "F.Paste")
-			(net "unconnected-(U1-IO2-Pad6)")
+			(net "/ESP32-S3/TMS")
 			(pinfunction "IO2_6")
 			(pintype "bidirectional")
@@
 			(size 0.8 0.4)
 			(layers "F.Cu" "F.Mask" "F.Paste")
-			(net "unconnected-(U1-IO3-Pad7)")
+			(net "/ESP32-S3/TDI")
 			(pinfunction "IO3_7")
 			(pintype "bidirectional")
@@
 			(size 0.8 0.4)
 			(layers "F.Cu" "F.Mask" "F.Paste")
-			(net "unconnected-(U1-IO4-Pad8)")
+			(net "/ESP32-S3/TDO")
 			(pinfunction "IO4_8")
 			(pintype "bidirectional")
